Commit message: feat(ros2): URDF 新增 imu_link 静态 TF（装配假设已注明）（任务 5/6）

File: ros2_car/src/robot_bringup/urdf/car.urdf (robot description, URDF)
Before this commit: robot car, 2 links, 1 joints
Links:
- added link imu_link
Joints:
- added joint imu_joint: type fixed, parent base_link, child imu_link, origin xyz=0.0 0.0 0.0 rpy=0 0 0
